File: Kicad_ERB_PEFAU_SCHERSACH/test/test.sch (KiCad schematic (older format))
At the start: 24 parts, among them J1 Conn_01x03, J2 Conn_01x03, J3 Conn_01x03, P1 Power, P2 Analog, P3 Digital, P4 Digital, P5 CONN_01X01, P6 CONN_01X01, P7 CONN_01X01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

Commit message: add kicad changes
Parts:
- C1, C2, C3: footprint Capacitor_SMD:CP_Elec_3x5.3 -> Capacitor_THT:C_Rect_L7.2mm_W3.0mm_P5.00mm_FKS2_FKP2_MKS2_MKP2
- C4: footprint Capacitor_SMD:CP_Elec_3x5.3 -> Capacitor_THT:C_Rect_L7.0mm_W6.0mm_P5.00mm
- J1, J2, J3: footprint Jumper:SolderJumper-3_P1.3mm_Bridged2Bar12_Pad1.0x1.5mm_NumberLabels -> Connector_PinHeader_2.54mm:PinHeader_1x03_P2.54mm_Vertical
- R1, R3, R5, R6, Rcal1, Rcal2: footprint Resistor_SMD:R_0201_0603Metric -> Resistor_THT:R_Axial_DIN0207_L6.3mm_D2.5mm_P10.16mm_Horizontal
Connections:
- net +3V3: no longer J1.2 (Pin_2)
- net +5V: now also J1.2 (Pin_2)
- net 8: now also U2.5 (RST)
- net A4(SDA): no longer P2.5 (Pin_5)
- net A5(SCL): no longer P2.6 (Pin_6)
- net 10: now reaches U2.1 (Tx)
- net 11: now reaches U2.2 (Rx)
- new net A4: P2.5 (Pin_5)
- new net A5: P2.6 (Pin_6)
Other:
- moved on the sheet: J1, J2, J3, U2
Changed lines of the file:
@@
 A3
 Text Label 8900 2900 0    60   ~ 0
-A4(SDA)
+A4
 Text Label 8900 3000 0    60   ~ 0
-A5(SCL)
+A5
 Text Label 10550 3000 0    60   ~ 0
 0(Rx)
@@
 $EndComp
 $Comp
-L My_Library:RN2483_Breakout U2
-U 1 1 5DD67E62
-P 1900 5250
-F 0 "U2" V 1954 5378 50  0000 L CNN
-F 1 "RN2483_Breakout" V 2045 5378 50  0000 L CNN
-F 2 "test:Module_RN2483" H 2000 5250 50  0001 C CNN
-F 3 "" H 2000 5250 50  0001 C CNN
-	1    1900 5250
-	0    -1   -1   0
-$EndComp
-$Comp
 L My_Library:Gaz_sensor U1
 U 1 1 5DE150DF
@@
 F 0 "Rcal1" H 3870 3996 50  0000 L CNN
 F 1 "33" H 3870 3905 50  0000 L CNN
-F 2 "Resistor_SMD:R_0201_0603Metric" V 3730 3950 50  0001 C CNN
+F 2 "Resistor_THT:R_Axial_DIN0207_L6.3mm_D2.5mm_P10.16mm_Horizontal" V 3730 3950 50  0001 C CNN
 F 3 "~" H 3800 3950 50  0001 C CNN
 	1    3800 3950
@@
 F 0 "C3" H 4865 2546 50  0000 L CNN
 F 1 "100n" H 4865 2455 50  0000 L CNN
-F 2 "Capacitor_SMD:CP_Elec_3x5.3" H 4788 2350 50  0001 C CNN
+F 2 "Capacitor_THT:C_Rect_L7.2mm_W3.0mm_P5.00mm_FKS2_FKP2_MKS2_MKP2" H 4788 2350 50  0001 C CNN
 F 3 "~" H 4750 2500 50  0001 C CNN
 	1    4750 2500
@@
 F 0 "Rcal2" H 3870 4496 50  0000 L CNN
 F 1 "33" H 3870 4405 50  0000 L CNN
-F 2 "Resistor_SMD:R_0201_0603Metric" V 3730 4450 50  0001 C CNN
+F 2 "Resistor_THT:R_Axial_DIN0207_L6.3mm_D2.5mm_P10.16mm_Horizontal" V 3730 4450 50  0001 C CNN
 F 3 "~" H 3800 4450 50  0001 C CNN
 	1    3800 4450
@@
 F 0 "R1" H 3370 3396 50  0000 L CNN
 F 1 "100k" H 3370 3305 50  0000 L CNN
-F 2 "Resistor_SMD:R_0201_0603Metric" V 3230 3350 50  0001 C CNN
+F 2 "Resistor_THT:R_Axial_DIN0207_L6.3mm_D2.5mm_P10.16mm_Horizontal" V 3230 3350 50  0001 C CNN
 F 3 "~" H 3300 3350 50  0001 C CNN
 	1    3300 3350
@@
 F 0 "R5" H 3020 2846 50  0000 L CNN
 F 1 "10k" H 3020 2755 50  0000 L CNN
-F 2 "Resistor_SMD:R_0201_0603Metric" V 2880 2800 50  0001 C CNN
+F 2 "Resistor_THT:R_Axial_DIN0207_L6.3mm_D2.5mm_P10.16mm_Horizontal" V 2880 2800 50  0001 C CNN
 F 3 "~" H 2950 2800 50  0001 C CNN
 	1    2950 2800
@@
 F 0 "C1" H 3065 3396 50  0000 L CNN
 F 1 "100n" H 3065 3305 50  0000 L CNN
-F 2 "Capacitor_SMD:CP_Elec_3x5.3" H 2988 3200 50  0001 C CNN
+F 2 "Capacitor_THT:C_Rect_L7.2mm_W3.0mm_P5.00mm_FKS2_FKP2_MKS2_MKP2" H 2988 3200 50  0001 C CNN
 F 3 "~" H 2950 3350 50  0001 C CNN
 	1    2950 3350
@@
 F 0 "C4" H 5365 3446 50  0000 L CNN
 F 1 "1µ" H 5365 3355 50  0000 L CNN
-F 2 "Capacitor_SMD:CP_Elec_3x5.3" H 5288 3250 50  0001 C CNN
+F 2 "Capacitor_THT:C_Rect_L7.0mm_W6.0mm_P5.00mm" H 5288 3250 50  0001 C CNN
 F 3 "~" H 5250 3400 50  0001 C CNN
 	1    5250 3400
@@
 F 0 "R3" H 5820 3446 50  0000 L CNN
 F 1 "100k" H 5820 3355 50  0000 L CNN
-F 2 "Resistor_SMD:R_0201_0603Metric" V 5680 3400 50  0001 C CNN
+F 2 "Resistor_THT:R_Axial_DIN0207_L6.3mm_D2.5mm_P10.16mm_Horizontal" V 5680 3400 50  0001 C CNN
 F 3 "~" H 5750 3400 50  0001 C CNN
 	1    5750 3400
@@
 F 0 "R6" V 6093 3150 50  0000 C CNN
 F 1 "1k" V 6184 3150 50  0000 C CNN
-F 2 "Resistor_SMD:R_0201_0603Metric" V 6230 3150 50  0001 C CNN
+F 2 "Resistor_THT:R_Axial_DIN0207_L6.3mm_D2.5mm_P10.16mm_Horizontal" V 6230 3150 50  0001 C CNN
 F 3 "~" H 6300 3150 50  0001 C CNN
 	1    6300 3150
@@
 F 0 "C2" H 6915 3446 50  0000 L CNN
 F 1 "100n" H 6915 3355 50  0000 L CNN
-F 2 "Capacitor_SMD:CP_Elec_3x5.3" H 6838 3250 50  0001 C CNN
+F 2 "Capacitor_THT:C_Rect_L7.2mm_W3.0mm_P5.00mm_FKS2_FKP2_MKS2_MKP2" H 6838 3250 50  0001 C CNN
 F 3 "~" H 6800 3400 50  0001 C CNN
 	1    6800 3400
@@
 L Connector_Generic:Conn_01x03 J1
 U 1 1 5DE76F5B
-P 1650 1900
-F 0 "J1" V 1522 2080 50  0000 L CNN
-F 1 "Conn_01x03" V 1613 2080 50  0000 L CNN
-F 2 "Jumper:SolderJumper-3_P1.3mm_Bridged2Bar12_Pad1.0x1.5mm_NumberLabels" H 1650 1900 50  0001 C CNN
-F 3 "~" H 1650 1900 50  0001 C CNN
-	1    1650 1900
+P 2800 1550
+F 0 "J1" V 2672 1730 50  0000 L CNN
+F 1 "Conn_01x03" V 2763 1730 50  0000 L CNN
+F 2 "Connector_PinHeader_2.54mm:PinHeader_1x03_P2.54mm_Vertical" H 2800 1550 50  0001 C CNN
+F 3 "~" H 2800 1550 50  0001 C CNN
+	1    2800 1550
 	0    1    1    0
 $EndComp
@@
 L Connector_Generic:Conn_01x03 J2
 U 1 1 5DE7F005
-P 2750 1950
-F 0 "J2" V 2622 2130 50  0000 L CNN
-F 1 "Conn_01x03" V 2713 2130 50  0000 L CNN
-F 2 "Jumper:SolderJumper-3_P1.3mm_Bridged2Bar12_Pad1.0x1.5mm_NumberLabels" H 2750 1950 50  0001 C CNN
-F 3 "~" H 2750 1950 50  0001 C CNN
-	1    2750 1950
+P 3900 1600
+F 0 "J2" V 3772 1780 50  0000 L CNN
+F 1 "Conn_01x03" V 3863 1780 50  0000 L CNN
+F 2 "Connector_PinHeader_2.54mm:PinHeader_1x03_P2.54mm_Vertical" H 3900 1600 50  0001 C CNN
+F 3 "~" H 3900 1600 50  0001 C CNN
+	1    3900 1600
 	0    1    1    0
 $EndComp
@@
 	1700 3400 1850 3400
 Wire Wire Line
-	1650 1500 1650 1700
-Text Label 1550 1550 0    50   ~ 0
+	2800 1150 2800 1350
+Text Label 2700 1200 0    50   ~ 0
 Gs_in
-Text Label 1750 1550 0    50   ~ 0
+Text Label 2900 1200 0    50   ~ 0
 Gs2_in
 Wire Wire Line
-	1550 1550 1550 1700
-Wire Wire Line
-	1750 1550 1750 1700
-Text Label 2650 1300 0    50   ~ 0
+	2700 1200 2700 1350
+Wire Wire Line
+	2900 1200 2900 1350
+Text Label 3800 950  0    50   ~ 0
 Gs1_out
-Text Label 2850 1400 0    50   ~ 0
+Text Label 4000 1050 0    50   ~ 0
 Gs2_out
-Text Label 2750 1550 0    50   ~ 0
+Text Label 3900 1200 0    50   ~ 0
 Rsensor
 Wire Wire Line
-	2650 1300 2650 1750
-Wire Wire Line
-	2750 1550 2750 1750
-Wire Wire Line
-	2850 1400 2850 1750
+	3800 950  3800 1400
+Wire Wire Line
+	3900 1200 3900 1400
+Wire Wire Line
+	4000 1050 4000 1400
 $Comp
 L power:+5V #PWR0111
@@
 L Connector_Generic:Conn_01x03 J3
 U 1 1 5DEACE77
-P 3800 1950
-F 0 "J3" V 3672 2130 50  0000 L CNN
-F 1 "Conn_01x03" V 3763 2130 50  0000 L CNN
-F 2 "Jumper:SolderJumper-3_P1.3mm_Bridged2Bar12_Pad1.0x1.5mm_NumberLabels" H 3800 1950 50  0001 C CNN
-F 3 "~" H 3800 1950 50  0001 C CNN
-	1    3800 1950
+P 4950 1600
+F 0 "J3" V 4822 1780 50  0000 L CNN
+F 1 "Conn_01x03" V 4913 1780 50  0000 L CNN
+F 2 "Connector_PinHeader_2.54mm:PinHeader_1x03_P2.54mm_Vertical" H 4950 1600 50  0001 C CNN
+F 3 "~" H 4950 1600 50  0001 C CNN
+	1    4950 1600
 	0    1    1    0
 $EndComp
@@
 L power:GND #PWR0113
 U 1 1 5DEADEC9
-P 3900 1500
-F 0 "#PWR0113" H 3900 1250 50  0001 C CNN
-F 1 "GND" H 3905 1327 50  0000 C CNN
-F 2 "" H 3900 1500 50  0001 C CNN
-F 3 "" H 3900 1500 50  0001 C CNN
-	1    3900 1500
+P 5050 1150
+F 0 "#PWR0113" H 5050 900 50  0001 C CNN
+F 1 "GND" H 5055 977 50  0000 C CNN
+F 2 "" H 5050 1150 50  0001 C CNN
+F 3 "" H 5050 1150 50  0001 C CNN
+	1    5050 1150
 	-1   0    0    1
 $EndComp
@@
 L power:+5V #PWR0114
 U 1 1 5DEAE74D
-P 3700 1500
-F 0 "#PWR0114" H 3700 1350 50  0001 C CNN
-F 1 "+5V" H 3715 1673 50  0000 C CNN
-F 2 "" H 3700 1500 50  0001 C CNN
-F 3 "" H 3700 1500 50  0001 C CNN
-	1    3700 1500
-	1    0    0    -1
-$EndComp
-Text Label 3800 1600 0    50   ~ 0
+P 4850 1150
+F 0 "#PWR0114" H 4850 1000 50  0001 C CNN
+F 1 "+5V" H 4865 1323 50  0000 C CNN
+F 2 "" H 4850 1150 50  0001 C CNN
+F 3 "" H 4850 1150 50  0001 C CNN
+	1    4850 1150
+	1    0    0    -1
+$EndComp
+Text Label 4950 1250 0    50   ~ 0
 Hr_in
 Wire Wire Line
-	3800 1600 3800 1750
-Wire Wire Line
-	3900 1500 3900 1750
-Wire Wire Line
-	3700 1500 3700 1750
-$Comp
-L power:GND #PWR?
+	4950 1250 4950 1400
+Wire Wire Line
+	5050 1150 5050 1400
+Wire Wire Line
+	4850 1150 4850 1400
+$Comp
+L power:+5V #PWR?
+U 1 1 5DF37CD9
+P 2800 1150
+F 0 "#PWR?" H 2800 1000 50  0001 C CNN
+F 1 "+5V" H 2815 1323 50  0000 C CNN
+F 2 "" H 2800 1150 50  0001 C CNN
+F 3 "" H 2800 1150 50  0001 C CNN
+	1    2800 1150
+	1    0    0    -1
+$EndComp
+Wire Wire Line
+	1750 1400 2000 1400
+Text Label 2000 1400 0    50   ~ 0
+8
+Wire Wire Line
+	1750 1700 2000 1700
+Text Label 2000 1700 0    50   ~ 0
+11
+Wire Wire Line
+	1750 1800 2000 1800
+Text Label 2000 1800 0    50   ~ 0
+10
+Wire Wire Line
+	1950 1300 1750 1300
+$Comp
+L power:+3V3 #PWR0115
+U 1 1 5DE777DB
+P 1950 1300
+F 0 "#PWR0115" H 1950 1150 50  0001 C CNN
+F 1 "+3V3" V 1965 1428 50  0000 L CNN
+F 2 "" H 1950 1300 50  0001 C CNN
+F 3 "" H 1950 1300 50  0001 C CNN
+	1    1950 1300
+	0    1    1    0
+$EndComp
+Wire Wire Line
+	1750 1100 1950 1100
+$Comp
+L power:GND #PWR0109
 U 1 1 5DE7110B
-P 2450 4800
-F 0 "#PWR?" H 2450 4550 50  0001 C CNN
-F 1 "GND" V 2455 4672 50  0000 R CNN
-F 2 "" H 2450 4800 50  0001 C CNN
-F 3 "" H 2450 4800 50  0001 C CNN
-	1    2450 4800
+P 1950 1100
+F 0 "#PWR0109" H 1950 850 50  0001 C CNN
+F 1 "GND" V 1955 972 50  0000 R CNN
+F 2 "" H 1950 1100 50  0001 C CNN
+F 3 "" H 1950 1100 50  0001 C CNN
+	1    1950 1100
 	0    -1   -1   0
 $EndComp
-Wire Wire Line
-	2250 4800 2450 4800
-$Comp
-L power:+3V3 #PWR?
-U 1 1 5DE76ED4
-P 1650 1500
-F 0 "#PWR?" H 1650 1350 50  0001 C CNN
-F 1 "+3V3" H 1665 1673 50  0000 C CNN
-F 2 "" H 1650 1500 50  0001 C CNN
-F 3 "" H 1650 1500 50  0001 C CNN
-	1    1650 1500
-	1    0    0    -1
-$EndComp
-$Comp
-L power:+3V3 #PWR?
-U 1 1 5DE777DB
-P 2500 5000
-F 0 "#PWR?" H 2500 4850 50  0001 C CNN
-F 1 "+3V3" V 2515 5128 50  0000 L CNN
-F 2 "" H 2500 5000 50  0001 C CNN
-F 3 "" H 2500 5000 50  0001 C CNN
-	1    2500 5000
-	0    1    1    0
-$EndComp
-Wire Wire Line
-	2250 5000 2500 5000
+$Comp
+L My_Library:RN2483_Breakout U2
+U 1 1 5DD67E62
+P 1400 1550
+F 0 "U2" V 1454 1678 50  0000 L CNN
+F 1 "RN2483_Breakout" V 1545 1678 50  0000 L CNN
+F 2 "test:Module_RN2483" H 1500 1550 50  0001 C CNN
+F 3 "" H 1500 1550 50  0001 C CNN
+	1    1400 1550
+	0    -1   -1   0
+$EndComp
 $EndSCHEMATC
